Commit message: added lidar supported plugins

File: urdf/accessories/rover_dev_payload.urdf (robot description, URDF)
Before this commit: robot rover_miti_payload, 1 links, 1 joints
Links:
- link payload_link: geometry collision mesh filename=file://$(find dummy_robot)/meshes/rover_payload.dae; visual mesh filename=file://$(find dummy_robot)/meshes/rover_payload.dae
